File: polarTRX.brd (EAGLE design)
At the start: 160 x 100 mm, 0 parts

Commit message: some parts added
Parts:
- added U1: PIC32MX250F128D, polarinstruments:TQFP44
- added U2: MAX4372, polarinstruments:SOT23-5DBV
- added U3: MCP1754S_SOT23, polarinstruments:SOT23
- added U4: LMP7702, polarinstruments:DGK_S-DPSO-G8
- added X1: USB+SHIELD, polarinstruments:USB-B-PTH
Connections:
- new net 1: U3.1
- new net 2: U3.2
- new net 3: U3.3
- new net P$1: U2.1
- new net P$3: U2.3
- new net V+: U4.8
- new net V-: U4.4
Changed lines of the file:
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@@
 </autorouter>
 <elements>
+<element name="U1" library="polarinstruments" package="TQFP44" value="PIC32MX250F128D" x="60.96" y="35.56"/>
+<element name="U2" library="polarinstruments" package="SOT23-5DBV" value="MAX4372" x="2.54" y="-3.81"/>
+<element name="X1" library="polarinstruments" package="USB-B-PTH" value="USB+SHIELD" x="10.16" y="-16.51"/>
+<element name="U3" library="polarinstruments" package="SOT23" value="MCP1754S_SOT23" x="2.54" y="-27.94"/>
+<element name="U4" library="polarinstruments" package="DGK_S-DPSO-G8" value="LMP7702" x="-3.81" y="-27.94"/>
 </elements>
 <signals>
+<signal name="P$1">
+<contactref element="U2" pad="1"/>
+</signal>
+<signal name="P$3">
+<contactref element="U2" pad="3"/>
+</signal>
+<signal name="1">
+<contactref element="U3" pad="1"/>
+</signal>
+<signal name="2">
+<contactref element="U3" pad="2"/>
+</signal>
+<signal name="3">
+<contactref element="U3" pad="3"/>
+</signal>
+<signal name="V+">
+<contactref element="U4" pad="8"/>
+</signal>
+<signal name="V-">
+<contactref element="U4" pad="4"/>
+</signal>
 </signals>
 </board>

Commit message: parts added
Parts:
- added C1: 10uF 16V, berry:C1206(3216)-A
- added C10: 1100pF, polarinstruments:C0603(1608)
- added C2, C3, C4, C5, C6, C7, C8: 0.1uF, polarinstruments:C0603(1608)
- added C9: 0.01uF, polarinstruments:C0603(1608)
- added JP1: (no value), SparkFun-Connectors:1X05
- added JP2: (no value), SparkFun-Connectors:1X03
- added R1: 0.5l, current sense, 0805, polarinstruments:R0805(2012)
- added R10, R9: 4.7k, polarinstruments:R0603(1608)
- added R2, R4, R5, R6, R7, R8: 10k, polarinstruments:R0603(1608)
- added R3: 1k, polarinstruments:R0603(1608)
- added S1, S2, S3, S4: (no value), polarinstruments:SKHLACA010
- added U5: LM94022, polarinstruments:SC70-5
- U2: value MAX4372 -> MAX4372F 50 Gain
- moved U1 105.1 mm to (-15.2, -36.8)
Connections:
- removed net 1: U3.1
- removed net 2: U3.2
- removed net 3: U3.3
- removed net P$1: U2.1
- removed net P$3: U2.3
- removed net V+: U4.8
- removed net V-: U4.4
- new net +3.3V: C1.1, JP1.2, R2.2, R4.2, R7.2, R8.2, U3.2
- new net +3.3V_ANALOG: C3.1, C8.1, C9.1, U2.3, U4.8, U5.4, U5.5
- new net AGND: C10.2, C3.2, C4.2, C5.2, C8.2, C9.2, U2.1, U4.4, U5.1, U5.2
- new net AN0: U4.1, U4.2
- new net AN1: U4.6, U4.7
- new net CURRENT_SENSE: R5.2, U2.2
- new net D+: X1.D+
- new net D-: X1.D-
- new net DGND: C1.2, C2.2, C6.2, C7.2, JP1.3, JP2.1, S2.P$2, S3.P$2, S4.P$2, U3.1, X1.GND
- new net N$1: R2.1, R3.2, S1.P$1
- new net N$10: C7.1, R8.1, S4.P$1
- new net N$11: R9.2, U1.34
- new net N$13: R6.2
- new net N$14: R10.2, U1.33
- new net N$2: C2.1, S1.P$2
- new net N$3: R1.2, U2.4, U3.3
- new net N$5: R1.1, U2.5
- new net N$7: C4.1, R5.1, U4.3
- new net N$8: C5.1, R6.1, U4.5
- new net N$9: C6.1, R7.1, S3.P$1
- new net PGEC: JP1.5, U1.22
- new net PGED: JP1.4, U1.21
- new net PRG: R4.1, S2.P$1, U1.32
- new net RESET: JP1.1, R3.1, U1.18
- new net RX: JP2.3, R9.1
- new net SCK: U1.15
- new net SDI: U1.1
- new net SDO: U1.4
- new net SS: U1.2
- new net STRUT_GND: X1.S1, X1.S2
- new net TEMP_SENSE: C10.1, U5.3
- new net TX: JP2.2, R10.1

Commit message: parts added
Parts:
- added C11, C12, C13, C14: 18pF, polarinstruments:C0603(1608)
- added Q1: (no value), polarinstruments:HC_49US
- added Q2: NX-3215, polarinstruments:NX-3215
- R1: value 0.5l, current sense, 0805 -> 0.51, current sense
- moved R1 199.3 mm to (-26.7, -233.7)
Connections:
- new net N$12: C14.1, Q2.1, U1.33
- new net N$15: R9.2, U1.26
- new net N$4: C11.1, Q1.3, U1.31
- new net N$6: C12.1, Q1.1, U1.30
- net DGND: now also C11.2, C12.2, C13.2, C14.2, Q1.2, U1.29, U1.39, U1.6
- net N$11: now also C13.1, Q2.2; no longer R9.2
- net N$14: now also U1.25; no longer U1.33
Changed lines of the file:
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@@
 <element name="U3" library="polarinstruments" package="SOT23" value="MCP1754S_SOT23" x="2.54" y="-27.94"/>
 <element name="U4" library="polarinstruments" package="DGK_S-DPSO-G8" value="LMP7702" x="-3.81" y="-27.94"/>
-<element name="R1" library="polarinstruments" package="R0805(2012)" value="0.5l, current sense, 0805" x="-5.08" y="-35.56"/>
 <element name="C1" library="berry" package="C1206(3216)-A" value="10uF 16V" x="-2.54" y="-41.91"/>
 <element name="U1" library="polarinstruments" package="TQFP44" value="PIC32MX250F128D" x="-15.24" y="-36.83"/>
@@
 <element name="C9" library="polarinstruments" package="C0603(1608)" value="0.01uF" x="-26.67" y="-181.61"/>
 <element name="C10" library="polarinstruments" package="C0603(1608)" value="1100pF" x="-26.67" y="-187.96"/>
+<element name="Q1" library="polarinstruments" package="HC_49US" value="" x="-20.32" y="-194.31"/>
+<element name="Q2" library="polarinstruments" package="NX-3215" value="NX-3215" x="-24.13" y="-204.47"/>
+<element name="C11" library="polarinstruments" package="C0603(1608)" value="18pF" x="-26.67" y="-208.28"/>
+<element name="C12" library="polarinstruments" package="C0603(1608)" value="18pF" x="-26.67" y="-214.63"/>
+<element name="C13" library="polarinstruments" package="C0603(1608)" value="18pF" x="-26.67" y="-220.98"/>
+<element name="C14" library="polarinstruments" package="C0603(1608)" value="18pF" x="-26.67" y="-227.33"/>
+<element name="R1" library="polarinstruments" package="R0805(2012)" value="0.51, current sense" x="-26.67" y="-233.68"/>
 </elements>
 <signals>
@@
 <contactref element="C6" pad="2"/>
 <contactref element="JP2" pad="1"/>
+<contactref element="U1" pad="29"/>
+<contactref element="U1" pad="39"/>
+<contactref element="U1" pad="6"/>
+<contactref element="Q1" pad="2"/>
+<contactref element="C11" pad="2"/>
+<contactref element="C12" pad="2"/>
+<contactref element="C14" pad="2"/>
+<contactref element="C13" pad="2"/>
+<wire x1="-25.92" y1="-220.98" x2="-25.92" y2="-227.33" width="0" layer="19" extent="1-1"/>
+<wire x1="-25.92" y1="-214.63" x2="-25.92" y2="-220.98" width="0" layer="19" extent="1-1"/>
+<wire x1="-25.92" y1="-208.28" x2="-25.92" y2="-214.63" width="0" layer="19" extent="1-1"/>
+<wire x1="-20.32" y1="-195.31" x2="-25.92" y2="-208.28" width="0" layer="19" extent="1-1"/>
+<wire x1="-19.05" y1="-153.67" x2="-20.32" y2="-195.31" width="0" layer="19" extent="1-1"/>
 <wire x1="-19.57" y1="-147.32" x2="-19.05" y2="-153.67" width="0" layer="19" extent="1-1"/>
 <wire x1="-19.57" y1="-140.97" x2="-19.57" y2="-147.32" width="0" layer="19" extent="1-1"/>
@@
 <wire x1="-13.26" y1="-71.12" x2="-13.97" y2="-110.49" width="0" layer="19" extent="1-1"/>
 <wire x1="-19.57" y1="-62.23" x2="-13.26" y2="-71.12" width="0" layer="19" extent="1-1"/>
-<wire x1="-1.24" y1="-41.91" x2="-19.57" y2="-62.23" width="0" layer="19" extent="1-1"/>
-<wire x1="1.59" y1="-29.04" x2="-1.24" y2="-41.91" width="0" layer="19" extent="1-1"/>
+<wire x1="-21.04" y1="-36.83" x2="-19.57" y2="-62.23" width="0" layer="19" extent="1-1"/>
+<wire x1="-15.24" y1="-31.03" x2="-21.04" y2="-36.83" width="0" layer="19" extent="1-1"/>
+<wire x1="-9.44" y1="-36.03" x2="-15.24" y2="-31.03" width="0" layer="19" extent="1-1"/>
+<wire x1="-1.24" y1="-41.91" x2="-9.44" y2="-36.03" width="0" layer="19" extent="1-1"/>
+<wire x1="1.59" y1="-29.04" x2="-9.44" y2="-36.03" width="0" layer="19" extent="1-1"/>
 <wire x1="12.8778" y1="-17.76" x2="1.59" y2="-29.04" width="0" layer="19" extent="1-1"/>
 </signal>
@@
 </signal>
 <signal name="N$3">
-<contactref element="R1" pad="2"/>
 <contactref element="U3" pad="3"/>
 <contactref element="U2" pad="4"/>
-<wire x1="2.54" y1="-26.84" x2="-4.13" y2="-35.56" width="0" layer="19" extent="1-1"/>
+<contactref element="R1" pad="2"/>
 <wire x1="3.49" y1="-2.51" x2="2.54" y2="-26.84" width="0" layer="19" extent="1-1"/>
+<wire x1="-25.72" y1="-233.68" x2="2.54" y2="-26.84" width="0" layer="19" extent="1-1"/>
 </signal>
 <signal name="N$5">
 <contactref element="U2" pad="5"/>
 <contactref element="R1" pad="1"/>
-<wire x1="1.59" y1="-2.51" x2="-6.03" y2="-35.56" width="0" layer="19" extent="1-1"/>
+<wire x1="1.59" y1="-2.51" x2="-27.62" y2="-233.68" width="0" layer="19" extent="1-1"/>
 </signal>
 <signal name="N$1">
@@
 <wire x1="-13.97" y1="-153.67" x2="-21.07" y2="-158.75" width="0" layer="19" extent="1-1"/>
 </signal>
-<signal name="N$11">
-<contactref element="U1" pad="34"/>
-<contactref element="R9" pad="2"/>
-<wire x1="-11.24" y1="-31.03" x2="-19.57" y2="-158.75" width="0" layer="19" extent="1-1"/>
-</signal>
-<signal name="N$14">
-<contactref element="U1" pad="33"/>
-<contactref element="R10" pad="2"/>
-<wire x1="-9.44" y1="-32.83" x2="-19.57" y2="-165.1" width="0" layer="19" extent="1-1"/>
-</signal>
 <signal name="CURRENT_SENSE">
 <contactref element="U2" pad="2"/>
@@
 <wire x1="-24.75" y1="-168.49" x2="-27.42" y2="-187.96" width="0" layer="19" extent="1-1"/>
 </signal>
+<signal name="N$4">
+<contactref element="U1" pad="31"/>
+<contactref element="Q1" pad="3"/>
+<contactref element="C11" pad="1"/>
+<wire x1="-16.02" y1="-194.31" x2="-27.42" y2="-208.28" width="0" layer="19" extent="1-1"/>
+<wire x1="-9.44" y1="-34.43" x2="-16.02" y2="-194.31" width="0" layer="19" extent="1-1"/>
+</signal>
+<signal name="N$6">
+<contactref element="U1" pad="30"/>
+<contactref element="Q1" pad="1"/>
+<contactref element="C12" pad="1"/>
+<wire x1="-24.62" y1="-194.31" x2="-27.42" y2="-214.63" width="0" layer="19" extent="1-1"/>
+<wire x1="-9.44" y1="-35.23" x2="-24.62" y2="-194.31" width="0" layer="19" extent="1-1"/>
+</signal>
+<signal name="N$11">
+<contactref element="U1" pad="34"/>
+<contactref element="Q2" pad="2"/>
+<contactref element="C13" pad="1"/>
+<wire x1="-22.88" y1="-204.47" x2="-27.42" y2="-220.98" width="0" layer="19" extent="1-1"/>
+<wire x1="-11.24" y1="-31.03" x2="-22.88" y2="-204.47" width="0" layer="19" extent="1-1"/>
+</signal>
+<signal name="N$12">
+<contactref element="U1" pad="33"/>
+<contactref element="Q2" pad="1"/>
+<contactref element="C14" pad="1"/>
+<wire x1="-25.38" y1="-204.47" x2="-27.42" y2="-227.33" width="0" layer="19" extent="1-1"/>
+<wire x1="-9.44" y1="-32.83" x2="-25.38" y2="-204.47" width="0" layer="19" extent="1-1"/>
+</signal>
+<signal name="N$14">
+<contactref element="R10" pad="2"/>
+<contactref element="U1" pad="25"/>
+<wire x1="-9.44" y1="-39.23" x2="-19.57" y2="-165.1" width="0" layer="19" extent="1-1"/>
+</signal>
+<signal name="N$15">
+<contactref element="R9" pad="2"/>
+<contactref element="U1" pad="26"/>
+<wire x1="-9.44" y1="-38.43" x2="-19.57" y2="-158.75" width="0" layer="19" extent="1-1"/>
+</signal>
 </signals>

Commit message: parts added
Parts:
- added C15, C18, C19, C20, C21: 0.1uF, polarinstruments:C0603(1608)
- added C16: 10uF 16V, berry:C1206(3216)-A
- added C17: 1uF 0805, polarinstruments:C0805(2012)
- added C22: 10uF 0805, polarinstruments:C0805(2012)
- added C23: 0.01uF, polarinstruments:C0603(1608)
- added L1: (no value), polarinstruments:L0805(2012)
- added LED1: 3mm, SparkFun-LED:LED3MM
- added LED2: 0603, SparkFun:LED-0603
- added R11: 10k, polarinstruments:R0603(1608)
- added TVS1: SD0, polarinstruments:SOD-323-NOPOL
Connections:
- new net +5V_USB: C23.1, R1.1, TVS1.2, U1.42, U2.5, X1.VBUS
- new net LED1: U1.12
- new net N$16: R11.2, U1.41
- net +3.3V: now also C18.1, C19.1, C20.1, L1.1, R11.1, U1.10, U1.28, U1.40
- net +3.3V_ANALOG: now also C21.1, C22.1, L1.2, U1.17
- net AGND: now also U1.16
- net D+: now also U1.8
- net D-: now also U1.9
- net DGND: now also C15.2, C16.2, C17.2, C18.2, C19.2, C20.2, C21.2, C22.2, C23.2, TVS1.1
- net N$3: now also C17.1
- net N$5: now also C15.1, C16.1, U1.7; no longer R1.1, U2.5

Commit message: temt 6000
Parts:
- removed C5: 0.1uF, polarinstruments:C0603(1608)
- added LD1: TEMT6000X01, polarinstruments:TEMT6000-SEN
- added R12: 100, polarinstruments:R0603(1608)
- added R13: 100k, polarinstruments:R0603(1608)
- added R14: 1k, polarinstruments:R0603(1608)
- R6: value 10k -> 100k
- moved R6 238.8 mm to (-26.7, -330.2)
Connections:
- removed net N$13: R6.2
- new net N$17: LD1.EMITTER, R12.1, U4.5
- net +3.3V_ANALOG: now also LD1.COLLECTOR
- net AGND: now also R12.2, R14.2, R6.2; no longer C5.2
- net AN1: now also R13.2; no longer U4.6
- net N$8: now also R13.1, U4.6; no longer C5.1, U4.5
Changed lines of the file:
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@@
 <element name="C3" library="polarinstruments" package="C0603(1608)" value="0.1uF" x="-20.32" y="-78.74"/>
 <element name="R5" library="polarinstruments" package="R0603(1608)" value="10k" x="-20.32" y="-85.09"/>
-<element name="R6" library="polarinstruments" package="R0603(1608)" value="10k" x="-20.32" y="-91.44"/>
 <element name="C4" library="polarinstruments" package="C0603(1608)" value="0.1uF" x="-20.32" y="-97.79"/>
-<element name="C5" library="polarinstruments" package="C0603(1608)" value="0.1uF" x="-20.32" y="-104.14"/>
 <element name="JP1" library="SparkFun-Connectors" package="1X05" value="" x="-19.05" y="-110.49"/>
 <element name="R7" library="polarinstruments" package="R0603(1608)" value="10k" x="-20.32" y="-121.92"/>
@@
 <element name="TVS1" library="polarinstruments" package="SOD-323-NOPOL" value="SD0" x="-24.13" y="-308.61"/>
 <element name="C23" library="polarinstruments" package="C0603(1608)" value="0.01uF" x="-26.67" y="-314.96"/>
+<element name="LD1" library="polarinstruments" package="TEMT6000-SEN" value="TEMT6000X01" x="-25.4" y="-318.77"/>
+<element name="R12" library="polarinstruments" package="R0603(1608)" value="100" x="-26.67" y="-323.85"/>
+<element name="R6" library="polarinstruments" package="R0603(1608)" value="100k" x="-26.67" y="-330.2"/>
+<element name="R13" library="polarinstruments" package="R0603(1608)" value="100k" x="-26.67" y="-336.55"/>
+<element name="R14" library="polarinstruments" package="R0603(1608)" value="1k" x="-26.67" y="-342.9"/>
 </elements>
 <signals>
@@
 <contactref element="U4" pad="4"/>
 <contactref element="C3" pad="2"/>
-<contactref element="C5" pad="2"/>
 <contactref element="C4" pad="2"/>
 <contactref element="U2" pad="1"/>
@@
 <contactref element="C10" pad="2"/>
 <contactref element="U1" pad="16"/>
+<contactref element="R12" pad="2"/>
+<contactref element="R6" pad="2"/>
+<contactref element="R14" pad="2"/>
 <wire x1="-25.92" y1="-181.61" x2="-25.92" y2="-187.96" width="0" layer="19" extent="1-1"/>
 <wire x1="-25.92" y1="-175.26" x2="-25.92" y2="-181.61" width="0" layer="19" extent="1-1"/>
 <wire x1="-26.05" y1="-168.49" x2="-25.92" y2="-175.26" width="0" layer="19" extent="1-1"/>
 <wire x1="-25.4" y1="-168.49" x2="-26.05" y2="-168.49" width="0" layer="19" extent="1-1"/>
-<wire x1="-19.57" y1="-104.14" x2="-25.4" y2="-168.49" width="0" layer="19" extent="1-1"/>
-<wire x1="-19.57" y1="-97.79" x2="-19.57" y2="-104.14" width="0" layer="19" extent="1-1"/>
+<wire x1="-19.57" y1="-97.79" x2="-25.4" y2="-168.49" width="0" layer="19" extent="1-1"/>
 <wire x1="-19.57" y1="-78.74" x2="-19.57" y2="-97.79" width="0" layer="19" extent="1-1"/>
 <wire x1="-16.04" y1="-42.63" x2="-19.57" y2="-78.74" width="0" layer="19" extent="1-1"/>
 <wire x1="-2.835" y1="-30.14" x2="-16.04" y2="-42.63" width="0" layer="19" extent="1-1"/>
 <wire x1="1.59" y1="-5.11" x2="-2.835" y2="-30.14" width="0" layer="19" extent="1-1"/>
+<wire x1="-25.92" y1="-323.85" x2="-25.92" y2="-187.96" width="0" layer="19" extent="1-1"/>
+<wire x1="-25.92" y1="-330.2" x2="-25.92" y2="-323.85" width="0" layer="19" extent="1-1"/>
+<wire x1="-25.92" y1="-342.9" x2="-25.92" y2="-330.2" width="0" layer="19" extent="1-1"/>
 </signal>
 <signal name="+3.3V_ANALOG">
@@
 <contactref element="C21" pad="1"/>
 <contactref element="C22" pad="1"/>
+<contactref element="LD1" pad="COLLECTOR"/>
 <wire x1="-27.42" y1="-175.26" x2="-27.42" y2="-181.61" width="0" layer="19" extent="1-1"/>
 <wire x1="-26.05" y1="-166.79" x2="-27.42" y2="-175.26" width="0" layer="19" extent="1-1"/>
@@
 <wire x1="-27.42" y1="-288.29" x2="-25.67" y2="-259.08" width="0" layer="19" extent="1-1"/>
 <wire x1="-27.67" y1="-294.64" x2="-27.42" y2="-288.29" width="0" layer="19" extent="1-1"/>
+<wire x1="-23.54" y1="-318.76" x2="-27.67" y2="-294.64" width="0" layer="19" extent="1-1"/>
 <wire x1="-21.07" y1="-78.74" x2="-24.75" y2="-166.79" width="0" layer="19" extent="1-1"/>
 <wire x1="-15.24" y1="-42.63" x2="-21.07" y2="-78.74" width="0" layer="19" extent="1-1"/>
@@
 </signal>
 <signal name="AN1">
-<contactref element="U4" pad="6"/>
 <contactref element="U4" pad="7"/>
-<wire x1="-4.135" y1="-25.74" x2="-3.485" y2="-25.74" width="0" layer="19" extent="1-1"/>
+<contactref element="R13" pad="2"/>
+<wire x1="-4.135" y1="-25.74" x2="-25.92" y2="-336.55" width="0" layer="19" extent="1-1"/>
 </signal>
 <signal name="N$7">
@@
 <wire x1="-3.485" y1="-30.14" x2="-21.07" y2="-85.09" width="0" layer="19" extent="1-1"/>
 </signal>
-<signal name="N$8">
-<contactref element="R6" pad="1"/>
-<contactref element="U4" pad="5"/>
-<contactref element="C5" pad="1"/>
-<wire x1="-21.07" y1="-91.44" x2="-21.07" y2="-104.14" width="0" layer="19" extent="1-1"/>
-<wire x1="-2.835" y1="-25.74" x2="-21.07" y2="-91.44" width="0" layer="19" extent="1-1"/>
-</signal>
 <signal name="PGED">
 <contactref element="JP1" pad="4"/>
@@
 <wire x1="-21.07" y1="-134.62" x2="-21.07" y2="-147.32" width="0" layer="19" extent="1-1"/>
 <wire x1="-19.76" y1="-127" x2="-21.07" y2="-134.62" width="0" layer="19" extent="1-1"/>
-</signal>
-<signal name="N$13">
-<contactref element="R6" pad="2"/>
 </signal>
 <signal name="SCK">
@@
 <contactref element="U1" pad="12"/>
 </signal>
+<signal name="N$17">
+<contactref element="R12" pad="1"/>
+<contactref element="LD1" pad="EMITTER"/>
+<contactref element="U4" pad="5"/>
+<wire x1="-27.27" y1="-318.12" x2="-27.42" y2="-323.85" width="0" layer="19" extent="1-1"/>
+<wire x1="-2.835" y1="-25.74" x2="-27.27" y2="-318.12" width="0" layer="19" extent="1-1"/>
+</signal>
+<signal name="N$8">
+<contactref element="U4" pad="6"/>
+<contactref element="R13" pad="1"/>
+<contactref element="R6" pad="1"/>
+<wire x1="-27.42" y1="-330.2" x2="-27.42" y2="-336.55" width="0" layer="19" extent="1-1"/>
+<wire x1="-3.485" y1="-25.74" x2="-27.42" y2="-330.2" width="0" layer="19" extent="1-1"/>
+</signal>
 </signals>
