File: polarTRX.brd (EAGLE design)
At the start: 160 x 100 mm, 55 parts, among them Q2 NX-3215, U1 PIC32MX250F128D, U2 MAX4372F 50 Gain, U3 MCP1754S_SOT23, U4 LMP7702, U5 LM94022, X1 USB+SHIELD

Commit message: schematic almost done
Parts:
- removed S4: (no value), polarinstruments:SKHLACA010
- added C24, C5: 0.1uF, polarinstruments:C0603(1608)
- added H1, H2, H3, H4: MOUNT-PAD-ROUND3.2, yBrainDigital:3,2-PAD
- added JP3: (no value), SparkFun-Connectors:1X05
- added R15, R16, R17: 10k, polarinstruments:R0603(1608)
- added R18: 100, polarinstruments:R0603(1608)
- added R19: 100k DNP, polarinstruments:R0603(1608)
- added R20: 1k, polarinstruments:R0603(1608)
- added R21: 100k, polarinstruments:R0603(1608)
- C10: value 1100pF -> 12.5pF
- C11, C12: value 18pF -> 0.1uF
- C15: value 0.1uF -> 10uF 0805; device polarinstruments:C0603(1608) -> polarinstruments:C0805(2012)
- C16: value 10uF 16V -> 0.1uF; device berry:C1206(3216)-A -> polarinstruments:C0603(1608)
- C17: value 1uF 0805 -> 0.1uF; device polarinstruments:C0805(2012) -> yBrainDigital:C0603(1608)
- C19: value 0.1uF -> 1100pF
- C20, C3: value 0.1uF -> 0.01uF
- C22: value 10uF 0805 -> 0.1uF; device polarinstruments:C0805(2012) -> polarinstruments:C0603(1608)
- C23: value 0.01uF -> 0.1uF
- C6: value 0.1uF -> 1uF 0805; device polarinstruments:C0603(1608) -> polarinstruments:C0805(2012)
- C7: value 0.1uF -> 10uF 16V; device polarinstruments:C0603(1608) -> berry:C1206(3216)-A
- C9: value 0.01uF -> 12.5pF
- JP1: device SparkFun-Connectors:1X05 -> SparkFun-Connectors:1X03
- JP2: value (none) -> M12PTH; device SparkFun-Connectors:1X03 -> SparkFun-Connectors:1X12
- LED1: value 3mm -> 0603; device SparkFun-LED:LED3MM -> SparkFun:LED-0603
- Q1: value (none) -> NX-3215; device polarinstruments:HC_49US -> polarinstruments:NX-3215
- Q2: value NX-3215 -> (none); device polarinstruments:NX-3215 -> polarinstruments:HC_49US
- R1: value 0.51, current sense -> 1k; device polarinstruments:R0805(2012) -> polarinstruments:R0603(1608)
- R10: value 4.7k -> 1M; device polarinstruments:R0603(1608) -> yBrainDigital:R0603(1608)
- R11, R2, R5: value 10k -> 1k
- R12: value 100 -> 1k
- R13: value 100k -> 10k
- R4: value 10k -> 0.51, current sense; device polarinstruments:R0603(1608) -> polarinstruments:R0805(2012)
- R6: value 100k -> 4.7k
- R7: value 10k -> 4.7k
- R9: value 4.7k -> 100k
- U1: value PIC32MX250F128D -> MAX4372F 50 Gain; device polarinstruments:TQFP44 -> polarinstruments:SOT23-5DBV
- U2: value MAX4372F 50 Gain -> MCP1754S_SOT23; device polarinstruments:SOT23-5DBV -> polarinstruments:SOT23
- U3: value MCP1754S_SOT23 -> PIC32MX250F128D; device polarinstruments:SOT23 -> polarinstruments:TQFP44
- U4: value LMP7702 -> LM94022; device polarinstruments:DGK_S-DPSO-G8 -> polarinstruments:SC70-5
- U5: value LM94022 -> LMP7702; device polarinstruments:SC70-5 -> polarinstruments:DGK_S-DPSO-G8
- moved R12 419.1 mm to (142.2, 59.7), turned to 90 degrees
- moved LED2 404.0 mm to (142.2, 63.5), turned to 180 degrees
- moved LED1 399.0 mm to (139.7, 63.5), turned to 180 degrees
- moved C22 397.9 mm to (120.7, 74.9), turned to 90 degrees
- moved R6 371.5 mm to (85.1, 24.1), turned to 180 degrees
- moved R14 356.0 mm to (19.1, 10.2), turned to 270 degrees
- moved R11 354.0 mm to (139.7, 59.7), turned to 90 degrees
- moved TVS1 350.3 mm to (16.5, 39.4), turned to 90 degrees
- moved C17 349.4 mm to (5.08, 85.1), turned to 90 degrees
- moved R13 347.2 mm to (19.1, 7.62), turned to 270 degrees
- moved L1 324.0 mm to (54.6, 54.6)
- moved C20 321.1 mm to (106.7, 10.2), turned to 180 degrees
- moved LD1 320.9 mm to (78.7, -15.2), turned to 180 degrees
- moved C19 316.6 mm to (104.1, 12.7), turned to 90 degrees
- moved C21 304.6 mm to (34.3, 10.2), turned to 90 degrees
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Connections:
- removed net N$17: LD1.EMITTER, R12.1, U4.5
- removed net N$7: C4.1, R5.1, U4.3
- removed net N$8: R13.1, R6.1, U4.6
- new net LED2: LED2.A, U3.44
- new net N$13: R1.2, U3.14
- new net N$18: LED1.C, R11.2
- new net N$19: LED2.C, R12.2
- new net N$20: R5.2, U3.1
- new net N$21: C23.1, R17.1, U5.3
- new net N$22: LD1.EMITTER, R18.1, U5.5
- new net N$23: R19.1, R20.1, R21.1, U5.6
- new net RF_GP0: JP2.12
- new net RF_GP1: JP2.11, R1.1
- new net RF_GP2: JP2.5
- new net RF_GP3: JP2.4, R3.1
- new net RF_NIRQ: JP2.10, R2.1
- new net RF_SDN: JP2.3, R5.1, R9.2
- new net SW1: C22.1, R16.1, S3.P$1, U3.43
- net +3.3V: now also C11.1, C12.1, C4.1, C7.1, C8.1, JP2.1, JP3.2, R13.2, R15.2, R16.2, R8.1, R9.1, U2.2, U3.10, U3.28, U3.40; no longer C1.1, C18.1, C19.1, C20.1, JP1.2, R11.1, R2.2, R4.2, R7.2, R8.2, U1.10, U1.28, U1.40, U3.2
- net +3.3V_ANALOG: now also C15.1, C16.1, C20.1, C24.1, C5.1, U1.3, U3.17, U4.4, U4.5, U5.8; no longer C21.1, C22.1, C3.1, C8.1, C9.1, U1.17, U2.3, U4.8, U5.4, U5.5
- net +5V_USB: now also C3.1, R4.1, U1.5, U3.42; no longer C23.1, R1.1, U1.42, U2.5
- net AGND: now also C19.2, C20.2, C23.2, C24.2, C5.2, R18.2, R19.2, R20.2, U1.1, U3.16, U4.1, U4.2, U5.4; no longer C10.2, C3.2, C4.2, C8.2, C9.2, R12.2, R14.2, R6.2, U1.16, U2.1, U4.4, U5.1, U5.2
- net AN0: now also U3.19, U5.1, U5.2; no longer U4.1, U4.2
- net AN1: now also R21.2, U3.20, U5.7; no longer R13.2, U4.7
- net CURRENT_SENSE: now also R17.2, U1.2; no longer R5.2, U2.2
- net D+: now also U3.8; no longer U1.8
- net D-: now also U3.9; no longer U1.9
- net DGND: now also C10.2, C17.1, C3.2, C4.2, C8.2, C9.2, JP1.1, JP2.2, JP3.3, Q2.2, R10.2, R11.1, R12.1, U2.1, U3.29, U3.39, U3.6; no longer C17.2, C19.2, C20.2, C23.2, JP1.3, JP2.1, Q1.2, S4.P$2, U1.29, U1.39, U1.6, U3.1
- net LED1: now also LED1.A, U3.12; no longer U1.12
- net N$1: now also R13.1, R14.2; no longer R2.1, R3.2
- net N$10: now also R3.2, U3.13; no longer C7.1, R8.1, S4.P$1
- net N$11: now also C9.1, Q1.2, U3.34; no longer C13.1, Q2.2, U1.34
- net N$12: now also C10.1, Q1.1, U3.33; no longer C14.1, Q2.1, U1.33
- net N$14: now also R7.2, U3.25; no longer R10.2, U1.25
- net N$15: now also R6.2, U3.26; no longer R9.2, U1.26
- net N$16: now also R8.2, U3.41; no longer R11.2, U1.41
- net N$2: now also C18.1; no longer C2.1
- net N$3: now also C6.1, R4.2, U1.4, U2.3; no longer C17.1, R1.2, U2.4, U3.3
- net N$4: now also C13.1, Q2.3, U3.31; no longer C11.1, Q1.3, U1.31
- net N$5: now also C1.1, C2.1, U3.7; no longer C15.1, C16.1, U1.7
- net N$6: now also C14.1, Q2.1, U3.30; no longer C12.1, Q1.1, U1.30
- net N$9: now also R2.2, U3.11; no longer C6.1, R7.1, S3.P$1
- net PGEC: now also JP3.5, U3.22; no longer JP1.5, U1.22
- net PGED: now also JP3.4, U3.21; no longer JP1.4, U1.21
- net PRG: now also C21.1, R15.1, U3.32; no longer R4.1, U1.32
- net RESET: now also JP3.1, R14.1, U3.18; no longer JP1.1, R3.1, U1.18
- net RX: now also JP1.3, R6.1; no longer JP2.3, R9.1
- net SCK: now also JP2.9, U3.15; no longer U1.15
- net SDI: now also JP2.8, U3.2; no longer U1.1
- net SDO: now also JP2.7, U3.4; no longer U1.4
- net SS: now also JP2.6, U3.5; no longer U1.2
- net STRUT_GND: now also C17.2, H1.B3,2, R10.1
- net TEMP_SENSE: now also C19.1, U3.23, U4.3; no longer C10.1, U5.3
- net TX: now also JP1.2, R7.1; no longer JP2.2, R10.1

Commit message: board layout done
Parts:
- added C25, C26, C27: 0.1uF, polarinstruments:C0603(1608)
- C17: device yBrainDigital:C0603(1608) -> polarinstruments:C0603(1608)
- C18: value 0.1uF -> 10uF 0805; device polarinstruments:C0603(1608) -> polarinstruments:C0805(2012)
- C19: value 1100pF -> 10uF 16V; device polarinstruments:C0603(1608) -> berry:C1206(3216)-A
- C20: value 0.01uF -> 0.1uF; device polarinstruments:C0603(1608) -> yBrainDigital:C0603(1608)
- C22: value 0.1uF -> 1100pF
- C23: value 0.1uF -> 0.01uF
- moved C17 111.1 mm to (91.4, 15.2), turned to 270 degrees
- moved C20 104.6 mm to (7.62, 43.8)
- moved C22 101.0 mm to (43.2, 10.2), turned to 270 degrees
- moved LED2 99.9 mm to (43.2, 50.8)
- moved R12 99.9 mm to (43.2, 47.0)
- moved LED1 99.9 mm to (40.6, 50.8)
- moved R11 99.9 mm to (40.6, 47.0)
- moved C24 87.0 mm to (31.8, 49.5), turned to 90 degrees
- moved JP1 81.2 mm to (74.9, 5.08), turned to 0 degrees
- moved R17 74.4 mm to (17.8, 10.2)
- moved S3 74.3 mm to (54.6, 48.3)
- moved C18 68.6 mm to (88.9, 15.2), turned to 270 degrees
- moved R16 67.2 mm to (58.4, 47.0)
- moved U4 66.1 mm to (40.6, 10.2), turned to 90 degrees
- moved R18 65.5 mm to (21.6, 5.08), turned to 90 degrees
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Connections:
- net D+ renamed D_P
- net D- renamed D_N
- removed net AGND: C19.2, C20.2, C23.2, C24.2, C5.2, R18.2, R19.2, R20.2, U1.1, U3.16, U4.1, U4.2, U5.4
- removed net N$3: C6.1, R4.2, U1.4, U2.3
- new net N$7: C3.1, R4.1, TVS1.2, U1.5, X1.VBUS
- net +3.3V: now also C17.1, C18.1, C19.1
- net +3.3V_ANALOG: now also C23.1, C27.1; no longer C20.1, C24.1
- net +5V_USB: now also C6.1, R4.2, U1.4, U2.3; no longer C3.1, R4.1, TVS1.2, U1.5, X1.VBUS
- net DGND: now also C17.2, C19.2, C20.1, C23.2, C24.2, C25.2, C26.2, C27.2, C5.2, R18.2, R19.2, R20.2, U1.1, U3.16, U4.1, U4.2, U5.4; no longer C17.1
- net N$2: now also C21.1; no longer C18.1
- net N$21: now also C26.1; no longer C23.1
- net PRG: now also C24.1; no longer C21.1
- net STRUT_GND: now also C20.2; no longer C17.2
- net SW1: now also C25.1; no longer C22.1
- net TEMP_SENSE: now also C22.1; no longer C19.1
Routing:
- net +3.3V: track 0.00 -> 189.8 mm, vias 0 -> 6
- net +3.3V_ANALOG: track 0.00 -> 86.7 mm
- net RF_SDN: track 0.00 -> 80.5 mm, vias 0 -> 3
- net DGND: track 0.00 -> 76.3 mm, vias 0 -> 50
- net RESET: track 0.00 -> 74.8 mm, vias 0 -> 6
- net SS: track 0.00 -> 71.9 mm, vias 0 -> 5
- net RF_NIRQ: track 0.00 -> 69.7 mm, vias 0 -> 4
- net SDO: track 0.00 -> 65.7 mm, vias 0 -> 5
- net RF_GP1: track 0.00 -> 63.3 mm, vias 0 -> 5
- net SCK: track 0.00 -> 59.3 mm, vias 0 -> 5
- net SDI: track 0.00 -> 58.8 mm, vias 0 -> 4
- net AN0: track 0.00 -> 55.6 mm, vias 0 -> 4
- net RF_GP3: track 0.00 -> 54.8 mm, vias 0 -> 4
- net AN1: track 0.00 -> 47.7 mm, vias 0 -> 4
- net PRG: track 0.00 -> 45.6 mm, vias 0 -> 4
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- added copper zone on layer 1, net DGND
- added copper zone on layer 16, net DGND
- added copper zone on layer 1, net STRUT_GND
- added copper zone on layer 16, net STRUT_GND
Other:
- board size 160 x 100 mm -> 140 x 60 mm
- board text added: "13 Jan 2016"
- board text added: "433 - 460 MHz"
- board text added: "ANTARCTICA"
- board text added: "GMSK TRX COMMS Board Ver 1."
- board text added: "GND"
- board text added: "GP0"
- board text added: "GP1"
- board text added: "GP2"
- board text added: "GP3"
- board text added: "MISO"
- board text added: "MOSI"
- board text added: "NRQ"
- board text added: "NSEL"
- board text added: "PROGRAM"
- board text added: "RESET"
- board text added: "RST"
- board text added: "RX"
- board text added: "SCLK"
- board text added: "SDN"
- board text added: "TX"
- board text added: "USER"
- board text added: "VDD"

Commit message: gerber file added
Parts:
- added JP4: (no value), SparkFun-Connectors:1X05
- added LED3: 0603, SparkFun:LED-0603
- added R22: 100k, polarinstruments:R0603(1608)
- added TP1: (no value), polarinstruments:TP-13
- JP2: value M12PTH -> (none); device SparkFun-Connectors:1X12 -> SparkFun-Connectors:1X08
- JP3: value (none) -> M12PTH; device SparkFun-Connectors:1X05 -> SparkFun-Connectors:1X12
- R13, R15, R8: value 10k -> 1k
- R14: value 1k -> 10k
- R18: value 100 -> 10k
- R19: value 100k DNP -> 100
- R20: value 1k -> 100k DNP
- R21: value 100k -> 1k
- R3: value 1k -> 0.51, current sense; device polarinstruments:R0603(1608) -> polarinstruments:R0805(2012)
- R4: value 0.51, current sense -> 1k; device polarinstruments:R0805(2012) -> polarinstruments:R0603(1608)
- R5: value 1k -> 4.7k
- R7: value 4.7k -> 10k
- moved R17 53.9 mm to (57.1, 47.0)
- moved JP2 47.8 mm to (62.2, 50.8), turned to 0 degrees
- moved JP3 39.4 mm to (95.0, 16.0), turned to 90 degrees
- moved R8 37.5 mm to (90.8, 41.6)
- moved R3 31.4 mm to (19.1, 27.9), turned to 0 degrees
- moved R16 26.7 mm to (31.8, 47.0)
- moved R4 26.2 mm to (43.2, 38.1)
- moved R5 24.4 mm to (64.8, 26.7), turned to 180 degrees
- moved LED1 24.4 mm to (21.6, 35.6), turned to 270 degrees
- moved R13 21.6 mm to (43.2, 47.0), turned to 90 degrees
- moved R11 19.6 mm to (24.8, 35.6), turned to 180 degrees
- moved R7 18.9 mm to (52.1, 39.4)
- moved R15 10.5 mm to (21.6, 49.5)
- moved R19 9.16 mm to (21.6, 5.08), turned to 90 degrees
- moved R18 6.35 mm to (17.8, 10.2), turned to 270 degrees
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Connections:
- new net N$19: LED3.C, R13.2
- new net SCK1: JP2.4, U3.14
- new net SDI1: JP2.6, U3.35
- new net SDO1: JP2.5, U3.36
- new net SS1: JP2.7, U3.38
- net +3.3V: now also JP2.3, JP3.1, JP4.2, R14.2, R17.2, R7.1; no longer JP2.1, JP3.2, R13.2, R15.2, R8.1
- net +5V_USB: now also JP2.1, LED1.A, R3.2; no longer R4.2
- net AN1: now also R22.2; no longer R21.2
- net CURRENT_SENSE: now also R18.2; no longer R17.2
- net DGND: now also JP2.8, JP3.2, JP4.3, R13.1, R21.2, TP1.TP; no longer JP3.3, R18.2
- net LED1: now also LED2.A; no longer LED1.A
- net LED2: now also LED3.A; no longer LED2.A
- net N$1: now also R14.1, R15.2; no longer R13.1, R14.2
- net N$10: now also R2.2; no longer R3.2
- net N$13: now also R8.2, U3.37; no longer R1.2, U3.14
- net N$14: now also R6.2; no longer R7.2
- net N$15: now also R5.2; no longer R6.2
- net N$16: now also R7.2; no longer R8.2
- net N$20: now also R4.2; no longer R5.2
- net N$21: now also R18.1; no longer R17.1
- net N$22: now also R19.1; no longer R18.1
- net N$23: now also R22.1; no longer R19.1
- net N$7: now also R3.1; no longer R4.1
- net N$9: now also R1.2; no longer R2.2
- net PGEC: now also JP4.5; no longer JP3.5
- net PGED: now also JP4.4; no longer JP3.4
- net PRG: now also R16.1; no longer R15.1
- net RESET: now also JP4.1, R15.1; no longer JP3.1, R14.1
- net RF_GP0: now also JP3.12; no longer JP2.12
- net RF_GP1: now also JP3.11, R8.1; no longer JP2.11, R1.1
- net RF_GP2: now also JP3.5; no longer JP2.5
- net RF_GP3: now also JP3.4, R2.1; no longer JP2.4, R3.1
- net RF_NIRQ: now also JP3.10, R1.1; no longer JP2.10, R2.1
- net RF_SDN: now also JP3.3, R4.1; no longer JP2.3, R5.1
- net RX: now also R5.1; no longer R6.1
- net SCK: now also JP3.9; no longer JP2.9
- net SDI: now also JP3.8; no longer JP2.8
- net SDO: now also JP3.7; no longer JP2.7
- net SS: now also JP3.6; no longer JP2.6
- net SW1: now also R17.1; no longer R16.1
- net TX: now also R6.1; no longer R7.1
Routing:
- net RF_GP1: track 63.3 -> 3.51 mm, vias 5 -> 0
- net +5V_USB: track 44.9 -> 102.1 mm, vias 4 -> 9
- net SCK1: track 0.00 -> 42.3 mm, vias 0 -> 4
- net N$13: track 3.36 -> 39.0 mm, vias 0 -> 2
- net SS1: track 0.00 -> 35.4 mm, vias 0 -> 2
- net +3.3V: track 189.8 -> 223.2 mm, vias 6 -> 8
- net SDI1: track 0.00 -> 27.9 mm, vias 0 -> 2
- net SDO1: track 0.00 -> 25.9 mm, vias 0 -> 2
- net RF_SDN: track 80.5 -> 85.5 mm
- net N$19: track 0.00 -> 2.31 mm
- net SS: track 71.9 -> 70.1 mm
- net DGND: track 76.3 -> 77.6 mm, vias 50 -> 51
- net SDO: track 65.7 -> 64.8 mm
- net PRG: track 45.6 -> 46.3 mm
- net N$17: track 2.31 -> 1.68 mm
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Other:
- board text added: "3V"
- board text added: "5V"
- board text added: "G"
- board text added: "SCK"
- board text added: "SS"
