File: polarTRX.sch (EAGLE design)
At the start: 0 parts

Commit message: some parts added
Parts:
- added U1: PIC32MX250F128D, polarinstruments:PIC32MX250F128D
- added U2: MAX4372, polarinstruments:MAX4372
- added U3: MCP1754S_SOT23, polarinstruments:MCP1754S_SOT23
- added U4: LMP7702, polarinstruments:LMP7702
- added X1: USB+SHIELD, polarinstruments:USB+SHIELD
Changed lines of the file:
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@@
 <parts>
 <part name="FRAME5" library="frames" deviceset="DINA4_L" device=""/>
+<part name="U1" library="polarinstruments" deviceset="PIC32MX250F128D" device=""/>
+<part name="U2" library="polarinstruments" deviceset="MAX4372" device=""/>
+<part name="X1" library="polarinstruments" deviceset="USB+SHIELD" device=""/>
+<part name="U3" library="polarinstruments" deviceset="MCP1754S" device="_SOT23"/>
+<part name="U4" library="polarinstruments" deviceset="LMP7702" device=""/>
 </parts>
 <sheets>
@@
 <instance part="FRAME5" gate="G$1" x="0" y="0"/>
 <instance part="FRAME5" gate="G$2" x="162.56" y="0"/>
+<instance part="U1" gate="G$1" x="124.46" y="101.6"/>
+<instance part="U2" gate="G$1" x="198.12" y="152.4"/>
+<instance part="X1" gate="G$1" x="142.24" y="152.4"/>
+<instance part="U3" gate="G$1" x="111.76" y="160.02"/>
+<instance part="U4" gate="A" x="187.96" y="127"/>
+<instance part="U4" gate="B" x="226.06" y="127"/>
+<instance part="U4" gate="G$2" x="187.96" y="127"/>
 </instances>
 <busses>

Commit message: parts added
Parts:
- added C1: 10uF 16V, berry:C-TANTAL-A
- added C10: 1100pF, polarinstruments:C0603(1608)
- added C2, C3, C4, C5, C6, C7, C8: 0.1uF, polarinstruments:C0603(1608)
- added C9: 0.01uF, polarinstruments:C0603(1608)
- added JP1: (no value), SparkFun-Connectors:M05PTH
- added JP2: (no value), SparkFun-Connectors:M03PTH
- added R1: 0.5l, current sense, 0805, polarinstruments:R0805(2012)
- added R10, R9: 4.7k, polarinstruments:R0603(1608)
- added R2, R4, R5, R6, R7, R8: 10k, polarinstruments:R0603(1608)
- added R3: 1k, polarinstruments:R0603(1608)
- added S1, S2, S3, S4: (no value), polarinstruments:SWITCH
- added U5: LM94022, polarinstruments:LM94022
- U2: value MAX4372 -> MAX4372F 50 Gain
Connections:
- new net +3.3V: C1.+, JP1.2, R2.2, R4.2, R7.2, R8.2, U3.2
- new net +3.3V_ANALOG: C3.1, C8.1, C9.1, U2.P$3, U4G$2.V+, U5.P$4, U5.P$5
- new net AGND: C10.2, C3.2, C4.2, C5.2, C8.2, C9.2, U2.P$1, U4G$2.V-, U5.P$1, U5.P$2
- new net AN0: U4A.-IN, U4A.OUT
- new net AN1: U4B.-IN, U4B.OUT
- new net CURRENT_SENSE: R5.2, U2.P$2
- new net D+: X1.D+
- new net D-: X1.D-
- new net DGND: C1.-, C2.2, C6.2, C7.2, JP1.3, JP2.1, S2.P$2, S3.P$2, S4.P$2, U3.1, X1.GND
- new net N$1: R2.1, R3.2, S1.P$1
- new net N$10: C7.1, R8.1, S4.P$1
- new net N$11: R9.2, U1.SOSCO
- new net N$13: R6.2
- new net N$14: R10.2, U1.SOSCI
- new net N$2: C2.1, S1.P$2
- new net N$3: R1.2, U2.P$4, U3.3
- new net N$5: R1.1, U2.P$5
- new net N$7: C4.1, R5.1, U4A.+IN
- new net N$8: C5.1, R6.1, U4B.+IN
- new net N$9: C6.1, R7.1, S3.P$1
- new net PGEC: JP1.5, U1.PGEC1
- new net PGED: JP1.4, U1.PGED1
- new net PRG: R4.1, S2.P$1, U1.TDO
- new net RESET: JP1.1, R3.1, U1./MCLR
- new net RX: JP2.3, R9.1
- new net SCK: U1.AN9
- new net SDI: U1.RPB9
- new net SDO: U1.RPC8
- new net SS: U1.RPC6
- new net STRUT_GND: X1.S1, X1.S2
- new net TEMP_SENSE: C10.1, U5.P$3
- new net TX: JP2.2, R10.1

Commit message: parts added
Parts:
- added C11, C12, C13, C14: 18pF, polarinstruments:C0603(1608)
- added Q1: (no value), polarinstruments:CRYSTAL
- added Q2: NX-3215, polarinstruments:NX-3215
- R1: value 0.5l, current sense, 0805 -> 0.51, current sense
Connections:
- new net N$12: C14.1, Q2.1, U1.SOSCI
- new net N$15: R9.2, U1.AN7
- new net N$4: C11.1, Q1.3, U1.OSC2
- new net N$6: C12.1, Q1.1, U1.OSC1
- net DGND: now also C11.2, C12.2, C13.2, C14.2, Q1.2, U1.VSS1, U1.VSS2, U1.VSS3
- net N$11: now also C13.1, Q2.2; no longer R9.2
- net N$14: now also U1.AN6; no longer U1.SOSCI
Other:
- note added: "U1TX: RPC0, U1RX: RPC1"
- moved on the sheet: C1, JP2, R10, R9

Commit message: parts added
Parts:
- added C15, C18, C19, C20, C21: 0.1uF, polarinstruments:C0603(1608)
- added C16: 10uF 16V, berry:C-TANTAL-A
- added C17: 1uF 0805, polarinstruments:C0805(2012)
- added C22: 10uF 0805, polarinstruments:C0805(2012)
- added C23: 0.01uF, polarinstruments:C0603(1608)
- added L1: (no value), polarinstruments:L0805(2012)
- added LED1: 3mm, SparkFun-LED:LED3MM
- added LED2: 0603, SparkFun:LED0603
- added R11: 10k, polarinstruments:R0603(1608)
- added TVS1: SD0, polarinstruments:SD0
Connections:
- new net +5V_USB: C23.1, R1.1, TVS1.P$2, U1.VBUS, U2.P$5, X1.VBUS
- new net LED1: U1.PGED4
- new net N$16: R11.2, U1.RPB5
- net +3.3V: now also C18.1, C19.1, C20.1, L1.1, R11.1, U1.VDD1, U1.VDD2, U1.VUSB3V3
- net +3.3V_ANALOG: now also C21.1, C22.1, L1.2, U1.AVDD
- net AGND: now also U1.AVSS
- net D+: now also U1.PGED2
- net D-: now also U1.PGEC2
- net DGND: now also C15.2, C16.-, C17.2, C18.2, C19.2, C20.2, C21.2, C22.2, C23.2, TVS1.P$1
- net N$3: now also C17.1
- net N$5: now also C15.1, C16.+, U1.VCAP; no longer R1.1, U2.P$5
Other:
- note added: "VBUS: For Monitoring USB Voltage"
- moved on the sheet: R10, R9

Commit message: temt 6000
Parts:
- removed C5: 0.1uF, polarinstruments:C0603(1608)
- added LD1: TEMT6000X01, polarinstruments:TEMT6000X01
- added R12: 100, polarinstruments:R0603(1608)
- added R13: 100k, polarinstruments:R0603(1608)
- added R14: 1k, polarinstruments:R0603(1608)
- R6: value 10k -> 100k
Connections:
- removed net N$13: R6.2
- new net N$17: LD1.E1, R12.1, U4B.+IN
- net +3.3V_ANALOG: now also LD1.C1
- net AGND: now also R12.2, R14.2, R6.2; no longer C5.2
- net AN1: now also R13.2; no longer U4B.-IN
- net N$8: now also R13.1, U4B.-IN; no longer C5.1, U4B.+IN
Other:
- moved on the sheet: R6, U4B
Changed lines of the file:
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@@
 <part name="AGND2" library="polarinstruments" deviceset="AGND" device=""/>
 <part name="R5" library="polarinstruments" deviceset="R" device="0603(1608)" value="10k"/>
-<part name="R6" library="polarinstruments" deviceset="R" device="0603(1608)" value="10k"/>
 <part name="C4" library="polarinstruments" deviceset="C" device="0603(1608)" value="0.1uF"/>
-<part name="C5" library="polarinstruments" deviceset="C" device="0603(1608)" value="0.1uF"/>
 <part name="AGND3" library="polarinstruments" deviceset="AGND" device=""/>
-<part name="AGND4" library="polarinstruments" deviceset="AGND" device=""/>
 <part name="JP1" library="SparkFun-Connectors" deviceset="M05" device="PTH"/>
 <part name="+3.3V4" library="berry" deviceset="+3.3V" device=""/>
@@
 <part name="C23" library="polarinstruments" deviceset="C" device="0603(1608)" value="0.01uF"/>
 <part name="GND16" library="berry" deviceset="DGND" device=""/>
+<part name="LD1" library="polarinstruments" deviceset="TEMT6000" device="X01"/>
+<part name="R12" library="polarinstruments" deviceset="R" device="0603(1608)" value="100"/>
+<part name="+3.3V_ANALOG6" library="polarinstruments" deviceset="+3.3V_ANALOG" device=""/>
+<part name="AGND12" library="polarinstruments" deviceset="AGND" device=""/>
+<part name="AGND4" library="polarinstruments" deviceset="AGND" device=""/>
+<part name="R6" library="polarinstruments" deviceset="R" device="0603(1608)" value="100k"/>
+<part name="R13" library="polarinstruments" deviceset="R" device="0603(1608)" value="100k"/>
+<part name="R14" library="polarinstruments" deviceset="R" device="0603(1608)" value="1k"/>
 </parts>
 <sheets>
@@
 <instance part="U3" gate="G$1" x="104.14" y="157.48" rot="R180"/>
 <instance part="U4" gate="A" x="187.96" y="127"/>
-<instance part="U4" gate="B" x="187.96" y="93.98"/>
+<instance part="U4" gate="B" x="299.72" y="121.92"/>
 <instance part="U4" gate="G$2" x="187.96" y="127"/>
 <instance part="C1" gate="G$1" x="121.92" y="154.94"/>
@@
 <instance part="AGND2" gate="VR1" x="203.2" y="137.16" rot="R90"/>
 <instance part="R5" gate="G$1" x="160.02" y="129.54" rot="R180"/>
-<instance part="R6" gate="G$1" x="160.02" y="96.52" rot="R180"/>
 <instance part="C4" gate="G$1" x="170.18" y="124.46"/>
-<instance part="C5" gate="G$1" x="170.18" y="91.44"/>
 <instance part="AGND3" gate="VR1" x="170.18" y="114.3"/>
-<instance part="AGND4" gate="VR1" x="170.18" y="81.28"/>
 <instance part="JP1" gate="G$1" x="104.14" y="215.9"/>
 <instance part="+3.3V4" gate="G$1" x="154.94" y="238.76"/>
@@
 <instance part="C23" gate="G$1" x="43.18" y="149.86"/>
 <instance part="GND16" gate="1" x="53.34" y="129.54"/>
+<instance part="LD1" gate="G$1" x="279.4" y="132.08"/>
+<instance part="R12" gate="G$1" x="281.94" y="116.84" rot="R270"/>
+<instance part="+3.3V_ANALOG6" gate="G$1" x="281.94" y="139.7"/>
+<instance part="AGND12" gate="VR1" x="281.94" y="106.68"/>
+<instance part="AGND4" gate="VR1" x="289.56" y="83.82"/>
+<instance part="R6" gate="G$1" x="289.56" y="96.52" rot="R270"/>
+<instance part="R13" gate="G$1" x="304.8" y="109.22"/>
+<instance part="R14" gate="G$1" x="297.18" y="96.52" rot="R270"/>
 </instances>
 <busses>
@@
 </segment>
 <segment>
-<pinref part="AGND4" gate="VR1" pin="AGND"/>
-<pinref part="C5" gate="G$1" pin="2"/>
-<wire x1="170.18" y1="83.82" x2="170.18" y2="86.36" width="0.1524" layer="91"/>
-</segment>
-<segment>
 <pinref part="AGND3" gate="VR1" pin="AGND"/>
 <pinref part="C4" gate="G$1" pin="2"/>
@@
 <pinref part="AGND11" gate="VR1" pin="AGND"/>
 <wire x1="63.5" y1="40.64" x2="53.34" y2="40.64" width="0.1524" layer="91"/>
+</segment>
+<segment>
+<pinref part="R12" gate="G$1" pin="2"/>
+<pinref part="AGND12" gate="VR1" pin="AGND"/>
+<wire x1="281.94" y1="109.22" x2="281.94" y2="111.76" width="0.1524" layer="91"/>
+</segment>
+<segment>
+<pinref part="AGND4" gate="VR1" pin="AGND"/>
+<pinref part="R6" gate="G$1" pin="2"/>
+<wire x1="289.56" y1="86.36" x2="289.56" y2="88.9" width="0.1524" layer="91"/>
+<pinref part="R14" gate="G$1" pin="2"/>
+<wire x1="289.56" y1="88.9" x2="289.56" y2="91.44" width="0.1524" layer="91"/>
+<wire x1="289.56" y1="88.9" x2="297.18" y2="88.9" width="0.1524" layer="91"/>
+<wire x1="297.18" y1="88.9" x2="297.18" y2="91.44" width="0.1524" layer="91"/>
+<junction x="289.56" y="88.9"/>
 </segment>
 </net>
@@
 <junction x="251.46" y="162.56"/>
 </segment>
+<segment>
+<pinref part="LD1" gate="G$1" pin="C1"/>
+<pinref part="+3.3V_ANALOG6" gate="G$1" pin="+3.3V_ANALOG"/>
+<wire x1="281.94" y1="137.16" x2="281.94" y2="139.7" width="0.1524" layer="91"/>
+</segment>
 </net>
 <net name="AN0" class="0">
@@
 <net name="AN1" class="0">
 <segment>
-<pinref part="U4" gate="B" pin="-IN"/>
-<wire x1="180.34" y1="91.44" x2="177.8" y2="91.44" width="0.1524" layer="91"/>
-<wire x1="177.8" y1="91.44" x2="177.8" y2="83.82" width="0.1524" layer="91"/>
-<wire x1="177.8" y1="83.82" x2="198.12" y2="83.82" width="0.1524" layer="91"/>
-<wire x1="198.12" y1="83.82" x2="198.12" y2="93.98" width="0.1524" layer="91"/>
+<wire x1="312.42" y1="109.22" x2="312.42" y2="121.92" width="0.1524" layer="91"/>
 <pinref part="U4" gate="B" pin="OUT"/>
-<wire x1="198.12" y1="93.98" x2="195.58" y2="93.98" width="0.1524" layer="91"/>
-<wire x1="198.12" y1="93.98" x2="203.2" y2="93.98" width="0.1524" layer="91"/>
-<junction x="198.12" y="93.98"/>
-<label x="203.2" y="93.98" size="1.778" layer="95" xref="yes"/>
+<wire x1="312.42" y1="121.92" x2="307.34" y2="121.92" width="0.1524" layer="91"/>
+<wire x1="312.42" y1="121.92" x2="314.96" y2="121.92" width="0.1524" layer="91"/>
+<junction x="312.42" y="121.92"/>
+<label x="314.96" y="121.92" size="1.778" layer="95" xref="yes"/>
+<pinref part="R13" gate="G$1" pin="2"/>
+<wire x1="309.88" y1="109.22" x2="312.42" y2="109.22" width="0.1524" layer="91"/>
 </segment>
 </net>
@@
 <wire x1="170.18" y1="127" x2="170.18" y2="129.54" width="0.1524" layer="91"/>
 <junction x="170.18" y="129.54"/>
-</segment>
-</net>
-<net name="N$8" class="0">
-<segment>
-<pinref part="R6" gate="G$1" pin="1"/>
-<pinref part="U4" gate="B" pin="+IN"/>
-<wire x1="165.1" y1="96.52" x2="170.18" y2="96.52" width="0.1524" layer="91"/>
-<pinref part="C5" gate="G$1" pin="1"/>
-<wire x1="170.18" y1="96.52" x2="180.34" y2="96.52" width="0.1524" layer="91"/>
-<wire x1="170.18" y1="93.98" x2="170.18" y2="96.52" width="0.1524" layer="91"/>
-<junction x="170.18" y="96.52"/>
 </segment>
 </net>
@@
 <wire x1="185.42" y1="223.52" x2="195.58" y2="223.52" width="0.1524" layer="91"/>
 <label x="195.58" y="223.52" size="1.778" layer="95" xref="yes"/>
-</segment>
-</net>
-<net name="N$13" class="0">
-<segment>
-<pinref part="R6" gate="G$1" pin="2"/>
-<wire x1="154.94" y1="96.52" x2="149.86" y2="96.52" width="0.1524" layer="91"/>
-<label x="149.86" y="96.52" size="1.778" layer="95" rot="R180" xref="yes"/>
 </segment>
 </net>
@@
 </segment>
 </net>
+<net name="N$17" class="0">
+<segment>
+<pinref part="R12" gate="G$1" pin="1"/>
+<pinref part="LD1" gate="G$1" pin="E1"/>
+<wire x1="281.94" y1="121.92" x2="281.94" y2="124.46" width="0.1524" layer="91"/>
+<pinref part="U4" gate="B" pin="+IN"/>
+<wire x1="281.94" y1="124.46" x2="281.94" y2="127" width="0.1524" layer="91"/>
+<wire x1="292.1" y1="124.46" x2="281.94" y2="124.46" width="0.1524" layer="91"/>
+<junction x="281.94" y="124.46"/>
+</segment>
+</net>
+<net name="N$8" class="0">
+<segment>
+<pinref part="U4" gate="B" pin="-IN"/>
+<wire x1="292.1" y1="119.38" x2="289.56" y2="119.38" width="0.1524" layer="91"/>
+<wire x1="289.56" y1="119.38" x2="289.56" y2="109.22" width="0.1524" layer="91"/>
+<pinref part="R13" gate="G$1" pin="1"/>
+<wire x1="299.72" y1="109.22" x2="289.56" y2="109.22" width="0.1524" layer="91"/>
+<pinref part="R6" gate="G$1" pin="1"/>
+<wire x1="289.56" y1="101.6" x2="289.56" y2="109.22" width="0.1524" layer="91"/>
+<junction x="289.56" y="109.22"/>
+</segment>
+</net>

Commit message: schematic almost done
Parts:
- removed S4: (no value), polarinstruments:SWITCH
- added C24, C5: 0.1uF, polarinstruments:C0603(1608)
- added H1, H2, H3, H4: MOUNT-PAD-ROUND3.2, yBrainDigital:MOUNT-PAD-ROUND3.2
- added JP3: (no value), SparkFun-Connectors:M05PTH
- added R15, R16, R17: 10k, polarinstruments:R0603(1608)
- added R18: 100, polarinstruments:R0603(1608)
- added R19: 100k DNP, polarinstruments:R0603(1608)
- added R20: 1k, polarinstruments:R0603(1608)
- added R21: 100k, polarinstruments:R0603(1608)
- C10: value 1100pF -> 12.5pF
- C11, C12: value 18pF -> 0.1uF
- C15: value 0.1uF -> 10uF 0805; device polarinstruments:C0603(1608) -> polarinstruments:C0805(2012)
- C16: value 10uF 16V -> 0.1uF; device berry:C-TANTAL-A -> polarinstruments:C0603(1608)
- C17: value 1uF 0805 -> 0.1uF; device polarinstruments:C0805(2012) -> yBrainDigital:C0603(1608)
- C19: value 0.1uF -> 1100pF
- C20, C3: value 0.1uF -> 0.01uF
- C22: value 10uF 0805 -> 0.1uF; device polarinstruments:C0805(2012) -> polarinstruments:C0603(1608)
- C23: value 0.01uF -> 0.1uF
- C6: value 0.1uF -> 1uF 0805; device polarinstruments:C0603(1608) -> polarinstruments:C0805(2012)
- C7: value 0.1uF -> 10uF 16V; device polarinstruments:C0603(1608) -> berry:C-TANTAL-A
- C9: value 0.01uF -> 12.5pF
- JP1: device SparkFun-Connectors:M05PTH -> SparkFun-Connectors:M03PTH
- JP2: value (none) -> M12PTH; device SparkFun-Connectors:M03PTH -> SparkFun-Connectors:M12PTH
- LED1: value 3mm -> 0603; device SparkFun-LED:LED3MM -> SparkFun:LED0603
- Q1: value (none) -> NX-3215; device polarinstruments:CRYSTAL -> polarinstruments:NX-3215
- Q2: value NX-3215 -> (none); device polarinstruments:NX-3215 -> polarinstruments:CRYSTAL
- R1: value 0.51, current sense -> 1k; device polarinstruments:R0805(2012) -> polarinstruments:R0603(1608)
- R10: value 4.7k -> 1M; device polarinstruments:R0603(1608) -> yBrainDigital:R0603(1608)
- R11, R2, R5: value 10k -> 1k
- R12: value 100 -> 1k
- R13: value 100k -> 10k
- R4: value 10k -> 0.51, current sense; device polarinstruments:R0603(1608) -> polarinstruments:R0805(2012)
- R6: value 100k -> 4.7k
- R7: value 10k -> 4.7k
- R9: value 4.7k -> 100k
- U1: value PIC32MX250F128D -> MAX4372F 50 Gain; device polarinstruments:PIC32MX250F128D -> polarinstruments:MAX4372
- U2: value MAX4372F 50 Gain -> MCP1754S_SOT23; device polarinstruments:MAX4372 -> polarinstruments:MCP1754S_SOT23
- U3: value MCP1754S_SOT23 -> PIC32MX250F128D; device polarinstruments:MCP1754S_SOT23 -> polarinstruments:PIC32MX250F128D
- U4: value LMP7702 -> LM94022; device polarinstruments:LMP7702 -> polarinstruments:LM94022
- U5: value LM94022 -> LMP7702; device polarinstruments:LM94022 -> polarinstruments:LMP7702
Connections:
- removed net N$17: LD1.E1, R12.1, U4B.+IN
- removed net N$7: C4.1, R5.1, U4A.+IN
- removed net N$8: R13.1, R6.1, U4B.-IN
- new net LED2: LED2.A, U3.RPB8
- new net N$13: R1.2, U3.CVREFOUT
- new net N$18: LED1.C, R11.2
- new net N$19: LED2.C, R12.2
- new net N$20: R5.2, U3.RPB9
- new net N$21: C23.1, R17.1, U5A.+IN
- new net N$22: LD1.E1, R18.1, U5B.+IN
- new net N$23: R19.1, R20.1, R21.1, U5B.-IN
- new net RF_GP0: JP2.12
- new net RF_GP1: JP2.11, R1.1
- new net RF_GP2: JP2.5
- new net RF_GP3: JP2.4, R3.1
- new net RF_NIRQ: JP2.10, R2.1
- new net RF_SDN: JP2.3, R5.1, R9.2
- new net SW1: C22.1, R16.1, S3.P$1, U3.RPB7
- net +3.3V: now also C11.1, C12.1, C4.1, C7.+, C8.1, JP2.1, JP3.2, R13.2, R15.2, R16.2, R8.1, R9.1, U2.2, U3.VDD1, U3.VDD2, U3.VUSB3V3; no longer C1.+, C18.1, C19.1, C20.1, JP1.2, R11.1, R2.2, R4.2, R7.2, R8.2, U1.VDD1, U1.VDD2, U1.VUSB3V3, U3.2
- net +3.3V_ANALOG: now also C15.1, C16.1, C20.1, C24.1, C5.1, U1.P$3, U3.AVDD, U4.P$4, U4.P$5, U5G$2.V+; no longer C21.1, C22.1, C3.1, C8.1, C9.1, U1.AVDD, U2.P$3, U4G$2.V+, U5.P$4, U5.P$5
- net +5V_USB: now also C3.1, R4.1, U1.P$5, U3.VBUS; no longer C23.1, R1.1, U1.VBUS, U2.P$5
- net AGND: now also C19.2, C20.2, C23.2, C24.2, C5.2, R18.2, R19.2, R20.2, U1.P$1, U3.AVSS, U4.P$1, U4.P$2, U5G$2.V-; no longer C10.2, C3.2, C4.2, C8.2, C9.2, R12.2, R14.2, R6.2, U1.AVSS, U2.P$1, U4G$2.V-, U5.P$1, U5.P$2
- net AN0: now also U3.PGED3, U5A.-IN, U5A.OUT; no longer U4A.-IN, U4A.OUT
- net AN1: now also R21.2, U3.PGEC3, U5B.OUT; no longer R13.2, U4B.OUT
- net CURRENT_SENSE: now also R17.2, U1.P$2; no longer R5.2, U2.P$2
- net D+: now also U3.PGED2; no longer U1.PGED2
- net D-: now also U3.PGEC2; no longer U1.PGEC2
- net DGND: now also C10.2, C16.2, C17.1, C3.2, C4.2, C7.-, C8.2, C9.2, JP1.1, JP2.2, JP3.3, Q2.2, R10.2, R11.1, R12.1, U2.1, U3.VSS1, U3.VSS2, U3.VSS3; no longer C16.-, C17.2, C19.2, C20.2, C23.2, C7.2, JP1.3, JP2.1, Q1.2, S4.P$2, U1.VSS1, U1.VSS2, U1.VSS3, U3.1
- net LED1: now also LED1.A, U3.PGED4; no longer U1.PGED4
- net N$1: now also R13.1, R14.2; no longer R2.1, R3.2
- net N$10: now also R3.2, U3.PGEC4; no longer C7.1, R8.1, S4.P$1
- net N$11: now also C9.1, Q1.2, U3.SOSCO; no longer C13.1, Q2.2, U1.SOSCO
- net N$12: now also C10.1, Q1.1, U3.SOSCI; no longer C14.1, Q2.1, U1.SOSCI
- net N$14: now also R7.2, U3.AN6; no longer R10.2, U1.AN6
- net N$15: now also R6.2, U3.AN7; no longer R9.2, U1.AN7
- net N$16: now also R8.2, U3.RPB5; no longer R11.2, U1.RPB5
- net N$2: now also C18.1; no longer C2.1
- net N$3: now also C6.1, R4.2, U1.P$4, U2.3; no longer C17.1, R1.2, U2.P$4, U3.3
- net N$4: now also C13.1, Q2.3, U3.OSC2; no longer C11.1, Q1.3, U1.OSC2
- net N$5: now also C1.+, C2.1, U3.VCAP; no longer C15.1, C16.+, U1.VCAP
- net N$6: now also C14.1, Q2.1, U3.OSC1; no longer C12.1, Q1.1, U1.OSC1
- net N$9: now also R2.2, U3.AN11; no longer C6.1, R7.1, S3.P$1
- net PGEC: now also JP3.5, U3.PGEC1; no longer JP1.5, U1.PGEC1
- net PGED: now also JP3.4, U3.PGED1; no longer JP1.4, U1.PGED1
- net PRG: now also C21.1, R15.1, U3.TDO; no longer R4.1, U1.TDO
- net RESET: now also JP3.1, R14.1, U3./MCLR; no longer JP1.1, R3.1, U1./MCLR
- net RX: now also JP1.3, R6.1; no longer JP2.3, R9.1
- net SCK: now also JP2.9, U3.AN9; no longer U1.AN9
- net SDI: now also JP2.8, U3.RPC6; no longer U1.RPB9
- net SDO: now also JP2.7, U3.RPC8; no longer U1.RPC8
- net SS: now also JP2.6, U3.RPC9; no longer U1.RPC6
- net STRUT_GND: now also C17.2, H1.MOUNT, R10.1
- net TEMP_SENSE: now also C19.1, U3.AN4, U4.P$3; no longer C10.1, U5.P$3
- net TX: now also JP1.2, R7.1; no longer JP2.2, R10.1
Other:
- note added: "0"
- note added: "1k: 1-1000lux setting"
- note added: "2"
- note added: "26"
- note added: "27"
- note added: "29"
- note added: "3"
- note added: "30"
- note added: "4"
- note added: "5 - A5"
- note added: "6 - A6"
- note added: "9 - A9"
- moved on the sheet: C1, C10, C11, C12, C13, C14, C15, C17, C2, C3, C4, C6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

Commit message: board layout done
Parts:
- added C25, C26, C27: 0.1uF, polarinstruments:C0603(1608)
- C17: device yBrainDigital:C0603(1608) -> polarinstruments:C0603(1608)
- C18: value 0.1uF -> 10uF 0805; device polarinstruments:C0603(1608) -> polarinstruments:C0805(2012)
- C19: value 1100pF -> 10uF 16V; device polarinstruments:C0603(1608) -> berry:C-TANTAL-A
- C20: value 0.01uF -> 0.1uF; device polarinstruments:C0603(1608) -> yBrainDigital:C0603(1608)
- C22: value 0.1uF -> 1100pF
- C23: value 0.1uF -> 0.01uF
Connections:
- net D+ renamed D_P
- net D- renamed D_N
- removed net AGND: C19.2, C20.2, C23.2, C24.2, C5.2, R18.2, R19.2, R20.2, U1.P$1, U3.AVSS, U4.P$1, U4.P$2, U5G$2.V-
- removed net N$3: C6.1, R4.2, U1.P$4, U2.3
- new net N$7: C3.1, R4.1, TVS1.P$2, U1.P$5, X1.VBUS
- net +3.3V: now also C17.1, C18.1, C19.+
- net +3.3V_ANALOG: now also C23.1, C27.1; no longer C20.1, C24.1
- net +5V_USB: now also C6.1, R4.2, U1.P$4, U2.3; no longer C3.1, R4.1, TVS1.P$2, U1.P$5, X1.VBUS
- net DGND: now also C17.2, C19.-, C20.1, C23.2, C24.2, C25.2, C26.2, C27.2, C5.2, R18.2, R19.2, R20.2, U1.P$1, U3.AVSS, U4.P$1, U4.P$2, U5G$2.V-; no longer C17.1
- net N$2: now also C21.1; no longer C18.1
- net N$21: now also C26.1; no longer C23.1
- net PRG: now also C24.1; no longer C21.1
- net STRUT_GND: now also C20.2; no longer C17.2
- net SW1: now also C25.1; no longer C22.1
- net TEMP_SENSE: now also C22.1; no longer C19.1
Other:
- moved on the sheet: C17, C21, C22, C23, C24, C4
