File: polarTRX.sch (EAGLE design)
At the start: 71 parts, among them Q1 NX-3215, U1 MAX4372F 50 Gain, U2 MCP1754S_SOT23, U3 PIC32MX250F128D, U4 LM94022, U5 LMP7702, X1 USB+SHIELD

Commit message: gerber file added
Parts:
- added JP4: (no value), SparkFun-Connectors:M05PTH
- added LED3: 0603, SparkFun:LED0603
- added R22: 100k, polarinstruments:R0603(1608)
- added TP1: (no value), polarinstruments:TP
- JP2: value M12PTH -> (none); device SparkFun-Connectors:M12PTH -> SparkFun-Connectors:M08SILK_FEMALE_PTH
- JP3: value (none) -> M12PTH; device SparkFun-Connectors:M05PTH -> SparkFun-Connectors:M12PTH
- R13, R15, R8: value 10k -> 1k
- R14: value 1k -> 10k
- R18: value 100 -> 10k
- R19: value 100k DNP -> 100
- R20: value 1k -> 100k DNP
- R21: value 100k -> 1k
- R3: value 1k -> 0.51, current sense; device polarinstruments:R0603(1608) -> polarinstruments:R0805(2012)
- R4: value 0.51, current sense -> 1k; device polarinstruments:R0805(2012) -> polarinstruments:R0603(1608)
- R5: value 1k -> 4.7k
- R7: value 4.7k -> 10k
Connections:
- new net N$19: LED3.C, R13.2
- new net SCK1: JP2.4, U3.CVREFOUT
- new net SDI1: JP2.6, U3.TDI
- new net SDO1: JP2.5, U3.AN12
- new net SS1: JP2.7, U3.RPC5
- net +3.3V: now also JP2.3, JP3.1, JP4.2, R14.2, R17.2, R7.1; no longer JP2.1, JP3.2, R13.2, R15.2, R8.1
- net +5V_USB: now also JP2.1, LED1.A, R3.2; no longer R4.2
- net AN1: now also R22.2; no longer R21.2
- net CURRENT_SENSE: now also R18.2; no longer R17.2
- net DGND: now also JP2.8, JP3.2, JP4.3, R13.1, R21.2, TP1.TP; no longer JP3.3, R18.2
- net LED1: now also LED2.A; no longer LED1.A
- net LED2: now also LED3.A; no longer LED2.A
- net N$1: now also R14.1, R15.2; no longer R13.1, R14.2
- net N$10: now also R2.2; no longer R3.2
- net N$13: now also R8.2, U3.RPC4; no longer R1.2, U3.CVREFOUT
- net N$14: now also R6.2; no longer R7.2
- net N$15: now also R5.2; no longer R6.2
- net N$16: now also R7.2; no longer R8.2
- net N$20: now also R4.2; no longer R5.2
- net N$21: now also R18.1; no longer R17.1
- net N$22: now also R19.1; no longer R18.1
- net N$23: now also R22.1; no longer R19.1
- net N$7: now also R3.1; no longer R4.1
- net N$9: now also R1.2; no longer R2.2
- net PGEC: now also JP4.5; no longer JP3.5
- net PGED: now also JP4.4; no longer JP3.4
- net PRG: now also R16.1; no longer R15.1
- net RESET: now also JP4.1, R15.1; no longer JP3.1, R14.1
- net RF_GP0: now also JP3.12; no longer JP2.12
- net RF_GP1: now also JP3.11, R8.1; no longer JP2.11, R1.1
- net RF_GP2: now also JP3.5; no longer JP2.5
- net RF_GP3: now also JP3.4, R2.1; no longer JP2.4, R3.1
- net RF_NIRQ: now also JP3.10, R1.1; no longer JP2.10, R2.1
- net RF_SDN: now also JP3.3, R4.1; no longer JP2.3, R5.1
- net RX: now also R5.1; no longer R6.1
- net SCK: now also JP3.9; no longer JP2.9
- net SDI: now also JP3.8; no longer JP2.8
- net SDO: now also JP3.7; no longer JP2.7
- net SS: now also JP3.6; no longer JP2.6
- net SW1: now also R17.1; no longer R16.1
- net TX: now also R6.1; no longer R7.1
Other:
- moved on the sheet: LED1, LED2, R1, R11, R12, R13, R14, R15, R16, R17, R18, R19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
